Commit message: fix: update camera intrinsics and adjust model properties for slim TurtleBot3

File: vslam_description/urdf/gz_slim_tb3.sdf.xacro (robot description, xacro)
@@ -2,13 +2,19 @@
 <sdf version="1.6" xmlns:xacro="http://www.ros.org/wiki/xacro">
     <xacro:arg name="namespace" default=""/>
-    <!-- Slim TurtleBot3: burger width, waffle-pi height, lidar removed, forward
-         monocular camera. Forked from nav2_minimal_tb3_sim/urdf/gz_waffle.sdf.xacro.
-         Body is centred at x=0 (the stock -0.064 offset existed only to match the
-         waffle_base.dae mesh origin, and we use primitives). -->
+    <!-- TurtleBot3 Burger with the lidar removed and a forward monocular camera.
+         Geometry follows the official ROBOTIS model at
+         /opt/ros/jazzy/share/turtlebot3_gazebo/models/turtlebot3_burger/model.sdf
+         rather than being re-derived: wheels y=+/-0.08, wheel_cz 0.023,
+         base_joint z 0.010, single rear caster at x=-0.081.
+         "Burger width, waffle-pi height" needs no scaling - the Burger body is
+         0.14 tall once the lidar tower is gone, which is the waffle-pi height.
+         Meshes resolve via model://turtlebot3_common/..., so
+         turtlebot3_gazebo/models must be on GZ_SIM_RESOURCE_PATH. -->
     <xacro:property name="body_x" value="0.138"/>
     <xacro:property name="body_y" value="0.138"/>
     <xacro:property name="body_z" value="0.141"/>
-    <!-- wheel bottom sits at z=-0.010; body bottom is held just above it at 0.0035 -->
-    <xacro:property name="body_cz" value="0.074"/>
+    <!-- mesh origin offset, from the official burger model -->
+    <xacro:property name="body_ox" value="-0.032"/>
+    <xacro:property name="body_cz" value="0.0705"/>
     <xacro:property name="wheel_y" value="0.080"/>
     <xacro:property name="wheel_r" value="0.033"/>
@@ -18,8 +24,6 @@
       <link name="base_footprint"/>
       <link name="base_link">
-        <!-- centre of mass held behind the wheel axis so the robot rests on the
-             rear casters instead of tipping forward -->
-        <inertial>
-          <pose>-0.020 0 0.050 0 0 0</pose>
+        <inertial>
+          <pose>-0.032 0 0.070 0 0 0</pose>
           <inertia>
             <ixx>0.001</ixx>
@@ -33,5 +37,5 @@
         </inertial>
         <collision name="base_collision">
-          <pose>0 0 ${body_cz} 0 0 0</pose>
+          <pose>${body_ox} 0 ${body_cz} 0 0 0</pose>
           <geometry>
             <box>
@@ -41,13 +45,15 @@
         </collision>
         <visual name="base_visual">
-          <pose>0 0 ${body_cz} 0 0 0</pose>
-          <geometry>
-            <box>
-              <size>${body_x} ${body_y} ${body_z}</size>
-            </box>
+          <pose>${body_ox} 0 0 0 0 0</pose>
+          <geometry>
+            <mesh>
+              <uri>model://turtlebot3_common/meshes/bases/burger_base.stl</uri>
+              <scale>0.001 0.001 0.001</scale>
+            </mesh>
           </geometry>
           <material>
-            <ambient>0.2 0.2 0.24 1</ambient>
+            <ambient>0.15 0.15 0.17 1</ambient>
             <diffuse>0.25 0.27 0.32 1</diffuse>
+            <specular>0.1 0.1 0.1 1</specular>
           </material>
         </visual>
@@ -147,10 +153,10 @@
         </collision>
         <visual name="wheel_left_visual">
-          <pose>0.0 ${wheel_y} ${wheel_cz} -1.57 0 0</pose>
-          <geometry>
-            <cylinder>
-              <radius>${wheel_r}</radius>
-              <length>0.018</length>
-            </cylinder>
+          <pose>0.0 ${wheel_y} ${wheel_cz} 0 0 0</pose>
+          <geometry>
+            <mesh>
+              <uri>model://turtlebot3_common/meshes/wheels/left_tire.stl</uri>
+              <scale>0.001 0.001 0.001</scale>
+            </mesh>
           </geometry>
           <material>
@@ -204,10 +210,10 @@
         </collision>
         <visual name="wheel_right_visual">
-          <pose>0.0 -${wheel_y} ${wheel_cz} -1.57 0 0</pose>
-          <geometry>
-            <cylinder>
-              <radius>${wheel_r}</radius>
-              <length>0.018</length>
-            </cylinder>
+          <pose>0.0 -${wheel_y} ${wheel_cz} 0 0 0</pose>
+          <geometry>
+            <mesh>
+              <uri>model://turtlebot3_common/meshes/wheels/right_tire.stl</uri>
+              <scale>0.001 0.001 0.001</scale>
+            </mesh>
           </geometry>
           <material>
@@ -217,17 +223,16 @@
         </visual>
       </link>
-      <!-- casters pulled forward from the stock -0.177: the slim body ends at
-           x=-0.069, so the stock position would float behind the robot -->
-      <link name='caster_back_right_link'>
-        <pose>-0.050 -0.045 -0.004 0 0 0</pose>
-        <inertial>
-          <mass>0.001</mass>
-          <inertia>
-            <ixx>0.00001</ixx>
-            <ixy>0.000</ixy>
-            <ixz>0.000</ixz>
-            <iyy>0.00001</iyy>
-            <iyz>0.000</iyz>
-            <izz>0.00001</izz>
+      <!-- single rear caster, position taken from the official burger model -->
+      <link name='caster_back_link'>
+        <pose>-0.081 0 -0.004 -1.57 0 0</pose>
+        <inertial>
+          <mass>0.005</mass>
+          <inertia>
+            <ixx>0.001</ixx>
+            <ixy>0.000</ixy>
+            <ixz>0.000</ixz>
+            <iyy>0.001</iyy>
+            <iyz>0.000</iyz>
+            <izz>0.001</izz>
           </inertia>
         </inertial>
@@ -252,42 +257,10 @@
         </collision>
       </link>
-      <link name='caster_back_left_link'>
-        <pose>-0.050 0.045 -0.004 0 0 0</pose>
-        <inertial>
-          <mass>0.001</mass>
-          <inertia>
-            <ixx>0.00001</ixx>
-            <ixy>0.000</ixy>
-            <ixz>0.000</ixz>
-            <iyy>0.00001</iyy>
-            <iyz>0.000</iyz>
-            <izz>0.00001</izz>
-          </inertia>
-        </inertial>
-        <collision name='collision'>
-          <geometry>
-            <sphere>
-              <radius>0.005000</radius>
-            </sphere>
-          </geometry>
-          <surface>
-            <contact>
-              <ode>
-                <soft_cfm>0</soft_cfm>
-                <soft_erp>0.2</soft_erp>
-                <kp>1e+5</kp>
-                <kd>1</kd>
-                <max_vel>0.01</max_vel>
-                <min_depth>0.001</min_depth>
-              </ode>
-            </contact>
-          </surface>
-        </collision>
-      </link>
-      <!-- forward-facing monocular camera, centred on y. 480x480 @ 30 Hz.
-           fx = fy = (480/2) / tan(1.047/2) = 415.69, cx = cy = 240.
+      <!-- forward monocular camera, centred on y, at the height the lidar
+           tower used to occupy. 480x480 @ 30 Hz.
+           Measured intrinsics: fx = fy = 415.787, cx = cy = 240.
            These MUST stay in sync with vslam_slam/config/tb3.yaml. -->
       <link name="camera_link">
-        <pose>0.064 0 0.115 0 0 0</pose>
+        <pose>0.032 0 0.115 0 0 0</pose>
         <inertial>
           <pose>0 0 0 0 0 0</pose>
@@ -305,5 +278,5 @@
           <geometry>
             <box>
-              <size>0.008 0.090 0.022</size>
+              <size>0.012 0.060 0.020</size>
             </box>
           </geometry>
@@ -312,9 +285,9 @@
           <geometry>
             <box>
-              <size>0.008 0.090 0.022</size>
+              <size>0.012 0.060 0.020</size>
             </box>
           </geometry>
           <material>
-            <ambient>0.6 0.2 0.1 1</ambient>
+            <ambient>0.5 0.15 0.05 1</ambient>
             <diffuse>0.8 0.3 0.15 1</diffuse>
           </material>
@@ -361,21 +334,17 @@
         </axis>
       </joint>
-      <joint name='caster_back_right_joint' type='ball'>
-        <parent>base_link</parent>
-        <child>caster_back_right_link</child>
-      </joint>
-      <joint name='caster_back_left_joint' type='ball'>
-        <parent>base_link</parent>
-        <child>caster_back_left_link</child>
+      <joint name='caster_back_joint' type='ball'>
+        <parent>base_link</parent>
+        <child>caster_back_link</child>
       </joint>
       <joint name="imu_joint" type="fixed">
         <parent>base_link</parent>
         <child>imu_link</child>
-        <pose>0.0 0 0.068 0 0 0</pose>
+        <pose>-0.032 0 0.068 0 0 0</pose>
       </joint>
       <joint name="camera_joint" type="fixed">
         <parent>base_link</parent>
         <child>camera_link</child>
-        <pose>0.064 0 0.115 0 0 0</pose>
+        <pose>0.032 0 0.115 0 0 0</pose>
         <axis>
           <xyz>0 0 1</xyz>
@@ -395,8 +364,8 @@
         <max_angular_acceleration>2</max_angular_acceleration>
         <min_angular_acceleration>-2</min_angular_acceleration>
-        <max_linear_velocity>0.46</max_linear_velocity>
-        <min_linear_velocity>-0.46</min_linear_velocity>
-        <max_angular_velocity>1.9</max_angular_velocity>
-        <min_angular_velocity>-1.9</min_angular_velocity>
+        <max_linear_velocity>0.22</max_linear_velocity>
+        <min_linear_velocity>-0.22</min_linear_velocity>
+        <max_angular_velocity>2.84</max_angular_velocity>
+        <min_angular_velocity>-2.84</min_angular_velocity>
         <topic>$(arg namespace)/cmd_vel</topic>
         <odom_topic>$(arg namespace)/odom</odom_topic>

Commit message: feat: add TurtleBot3 burger base mesh and cutting script for simulation

File: vslam_description/urdf/gz_slim_tb3.sdf.xacro (robot description, xacro)
@@ -13,11 +13,24 @@
     <xacro:property name="body_x" value="0.138"/>
     <xacro:property name="body_y" value="0.138"/>
-    <xacro:property name="body_z" value="0.141"/>
+    <!-- Collision spans z 0.000..0.066 (cap plate top). It must NOT reach down
+         to the mesh bottom at -10mm: ground contact is at z=-0.010, so a box
+         that low scrapes the floor and physics shoves the robot around. -->
+    <xacro:property name="body_z" value="0.066"/>
     <!-- mesh origin offset, from the official burger model -->
     <xacro:property name="body_ox" value="-0.032"/>
-    <xacro:property name="body_cz" value="0.0705"/>
+    <xacro:property name="body_cz" value="0.033"/>
     <xacro:property name="wheel_y" value="0.080"/>
     <xacro:property name="wheel_r" value="0.033"/>
     <xacro:property name="wheel_cz" value="0.023"/>
+    <!-- deck1 mesh tops out at 60.5mm; the cap plate sits just above it -->
+    <xacro:property name="deck_z" value="0.063"/>
+    <xacro:property name="cam_z" value="0.115"/>
+    <xacro:property name="mast_x" value="0.010"/>
+    <!-- colour scheme -->
+    <xacro:property name="c_body" value="0.10 0.28 0.32"/>
+    <xacro:property name="c_body_amb" value="0.04 0.11 0.13"/>
+    <xacro:property name="c_accent" value="0.90 0.45 0.10"/>
+    <xacro:property name="c_accent_amb" value="0.35 0.16 0.03"/>
+    <xacro:property name="c_dark" value="0.13 0.14 0.16"/>
     <model name="slim_tb3">
       <pose>0.0 0.0 0.0 0.0 0.0 0.0</pose>
@@ -44,16 +57,57 @@
           </geometry>
         </collision>
+        <!-- Burger base plate only. Upper two decks cut off at z=62mm by
+             scripts/cut_stl.py; see meshes/README.md for regeneration. -->
         <visual name="base_visual">
           <pose>${body_ox} 0 0 0 0 0</pose>
           <geometry>
             <mesh>
-              <uri>model://turtlebot3_common/meshes/bases/burger_base.stl</uri>
+              <uri>package://vslam_description/meshes/burger_deck1.stl</uri>
               <scale>0.001 0.001 0.001</scale>
             </mesh>
           </geometry>
           <material>
-            <ambient>0.15 0.15 0.17 1</ambient>
-            <diffuse>0.25 0.27 0.32 1</diffuse>
+            <ambient>${c_body_amb} 1</ambient>
+            <diffuse>${c_body} 1</diffuse>
             <specular>0.1 0.1 0.1 1</specular>
+          </material>
+        </visual>
+        <!-- cap plate: closes the open top left by the mesh cut -->
+        <visual name="deck_plate_visual">
+          <pose>${body_ox} 0 ${deck_z} 0 0 0</pose>
+          <geometry>
+            <box>
+              <size>0.128 0.128 0.005</size>
+            </box>
+          </geometry>
+          <material>
+            <ambient>${c_accent_amb} 1</ambient>
+            <diffuse>${c_accent} 1</diffuse>
+          </material>
+        </visual>
+        <!-- camera mast -->
+        <visual name="mast_visual">
+          <pose>${mast_x} 0 ${(deck_z + cam_z) / 2} 0 0 0</pose>
+          <geometry>
+            <box>
+              <size>0.014 0.030 ${cam_z - deck_z}</size>
+            </box>
+          </geometry>
+          <material>
+            <ambient>0.05 0.05 0.06 1</ambient>
+            <diffuse>${c_dark} 1</diffuse>
+          </material>
+        </visual>
+        <!-- bracket arm from mast to camera -->
+        <visual name="mast_arm_visual">
+          <pose>${(mast_x + 0.032) / 2} 0 ${cam_z} 0 0 0</pose>
+          <geometry>
+            <box>
+              <size>0.030 0.024 0.008</size>
+            </box>
+          </geometry>
+          <material>
+            <ambient>0.05 0.05 0.06 1</ambient>
+            <diffuse>${c_dark} 1</diffuse>
           </material>
         </visual>
@@ -289,6 +343,6 @@
           </geometry>
           <material>
-            <ambient>0.5 0.15 0.05 1</ambient>
-            <diffuse>0.8 0.3 0.15 1</diffuse>
+            <ambient>${c_accent_amb} 1</ambient>
+            <diffuse>${c_accent} 1</diffuse>
           </material>
         </visual>

Commit message: fix: update vslam-sim documentation and adjust mesh properties for TurtleBot3 simulation

File: vslam_description/urdf/gz_slim_tb3.sdf.xacro (robot description, xacro)
@@ -23,6 +23,6 @@
     <xacro:property name="wheel_r" value="0.033"/>
     <xacro:property name="wheel_cz" value="0.023"/>
-    <!-- deck1 mesh tops out at 60.5mm; the cap plate sits just above it -->
-    <xacro:property name="deck_z" value="0.063"/>
+    <!-- deck1 mesh tops out at 60.5mm; the bracket stands directly on it -->
+    <xacro:property name="deck_z" value="0.060"/>
     <xacro:property name="cam_z" value="0.115"/>
     <xacro:property name="mast_x" value="0.010"/>
@@ -71,17 +71,4 @@
             <diffuse>${c_body} 1</diffuse>
             <specular>0.1 0.1 0.1 1</specular>
-          </material>
-        </visual>
-        <!-- cap plate: closes the open top left by the mesh cut -->
-        <visual name="deck_plate_visual">
-          <pose>${body_ox} 0 ${deck_z} 0 0 0</pose>
-          <geometry>
-            <box>
-              <size>0.128 0.128 0.005</size>
-            </box>
-          </geometry>
-          <material>
-            <ambient>${c_accent_amb} 1</ambient>
-            <diffuse>${c_accent} 1</diffuse>
           </material>
         </visual>

Commit message: feat: enhance navigation capabilities for TurtleBot3 with ORB-SLAM3 integration
- Updated bringup_sim.launch.py to include navigation launch configuration.
- Added vslam_navigation package with necessary launch files and parameters.
- Integrated LDS lidar into the simulation for Nav2 costmaps.
- Modified mono_slam_node to publish map to odom transformations.
- Updated CMakeLists.txt and package.xml to include new dependencies.

File: vslam_description/urdf/gz_slim_tb3.sdf.xacro (robot description, xacro)
@@ -74,4 +74,18 @@
         </visual>
         <!-- camera mast -->
+        <!-- post carrying the lidar above the camera bracket -->
+        <visual name="lidar_post_visual">
+          <pose>-0.032 0 ${(deck_z + 0.150) / 2} 0 0 0</pose>
+          <geometry>
+            <cylinder>
+              <radius>0.010</radius>
+              <length>${0.150 - deck_z}</length>
+            </cylinder>
+          </geometry>
+          <material>
+            <ambient>0.05 0.05 0.06 1</ambient>
+            <diffuse>${c_dark} 1</diffuse>
+          </material>
+        </visual>
         <visual name="mast_visual">
           <pose>${mast_x} 0 ${(deck_z + cam_z) / 2} 0 0 0</pose>
@@ -99,4 +113,68 @@
           </material>
         </visual>
+      </link>
+      <!-- LDS lidar for Nav2 costmaps. Mounted at z=0.150 on a post so it
+           clears the camera bracket (top at z=0.119) - a lower mount would
+           put the bracket in the scan and blind the robot forward. -->
+      <link name="base_scan">
+        <pose>-0.032 0 0.150 0 0 0</pose>
+        <inertial>
+          <inertia>
+            <ixx>0.001</ixx>
+            <ixy>0.000</ixy>
+            <ixz>0.000</ixz>
+            <iyy>0.001</iyy>
+            <iyz>0.000</iyz>
+            <izz>0.001</izz>
+          </inertia>
+          <mass>0.114</mass>
+        </inertial>
+        <collision name="lidar_collision">
+          <geometry>
+            <cylinder>
+              <radius>0.0508</radius>
+              <length>0.055</length>
+            </cylinder>
+          </geometry>
+        </collision>
+        <visual name="lidar_visual">
+          <geometry>
+            <mesh>
+              <uri>model://turtlebot3_common/meshes/sensors/lds.stl</uri>
+              <scale>0.001 0.001 0.001</scale>
+            </mesh>
+          </geometry>
+          <material>
+            <ambient>0.05 0.05 0.06 1</ambient>
+            <diffuse>${c_dark} 1</diffuse>
+          </material>
+        </visual>
+        <sensor name="hls_lfcd_lds" type="gpu_lidar">
+          <always_on>true</always_on>
+          <visualize>true</visualize>
+          <update_rate>10</update_rate>
+          <topic>scan</topic>
+          <gz_frame_id>base_scan</gz_frame_id>
+          <ray>
+            <scan>
+              <horizontal>
+                <samples>360</samples>
+                <resolution>1.000000</resolution>
+                <min_angle>0.000000</min_angle>
+                <max_angle>6.280000</max_angle>
+              </horizontal>
+            </scan>
+            <range>
+              <min>0.120000</min>
+              <max>3.5</max>
+              <resolution>0.015000</resolution>
+            </range>
+            <noise>
+              <type>gaussian</type>
+              <mean>0.0</mean>
+              <stddev>0.01</stddev>
+            </noise>
+          </ray>
+        </sensor>
       </link>
       <link name="imu_link">
@@ -379,4 +457,12 @@
         <child>caster_back_link</child>
       </joint>
+      <joint name="lidar_joint" type="fixed">
+        <parent>base_link</parent>
+        <child>base_scan</child>
+        <pose>-0.032 0 0.150 0 0 0</pose>
+        <axis>
+          <xyz>0 0 1</xyz>
+        </axis>
+      </joint>
       <joint name="imu_joint" type="fixed">
         <parent>base_link</parent>

Commit message: Refactor code structure for improved readability and maintainability

File: vslam_description/urdf/gz_slim_tb3.sdf.xacro (robot description, xacro)
@@ -25,5 +25,14 @@
     <!-- deck1 mesh tops out at 60.5mm; the bracket stands directly on it -->
     <xacro:property name="deck_z" value="0.060"/>
-    <xacro:property name="cam_z" value="0.115"/>
+    <!-- Raised from 0.115. At that height the optical axis was horizontal and
+         the bottom half of every frame was floor from ~0.2 m out - close,
+         low-parallax, repetitively textured, and a poor diet for monocular
+         tracking. At 0.25 with a 5 deg upward tilt the floor starts ~0.7 m out
+         and pillars/walls dominate the frame.
+         The lidar scan plane is at 0.150; the bracket crossing it sits 0.061 m
+         from the lidar, inside range_min 0.12, so it is not seen. -->
+    <xacro:property name="cam_z" value="0.250"/>
+    <!-- negative pitch = nose up in SDF -->
+    <xacro:property name="cam_pitch" value="-0.0873"/>
     <xacro:property name="mast_x" value="0.010"/>
     <!-- colour scheme -->
@@ -92,5 +101,5 @@
           <geometry>
             <box>
-              <size>0.014 0.030 ${cam_z - deck_z}</size>
+              <size>0.016 0.030 ${cam_z - deck_z}</size>
             </box>
           </geometry>
@@ -102,5 +111,5 @@
         <!-- bracket arm from mast to camera -->
         <visual name="mast_arm_visual">
-          <pose>${(mast_x + 0.032) / 2} 0 ${cam_z} 0 0 0</pose>
+          <pose>${(mast_x + 0.032) / 2} 0 ${cam_z} 0 ${cam_pitch} 0</pose>
           <geometry>
             <box>
@@ -381,5 +390,5 @@
            These MUST stay in sync with vslam_slam/config/tb3.yaml. -->
       <link name="camera_link">
-        <pose>0.032 0 0.115 0 0 0</pose>
+        <pose>0.032 0 ${cam_z} 0 ${cam_pitch} 0</pose>
         <inertial>
           <pose>0 0 0 0 0 0</pose>
@@ -473,5 +482,5 @@
         <parent>base_link</parent>
         <child>camera_link</child>
-        <pose>0.032 0 0.115 0 0 0</pose>
+        <pose>0.032 0 ${cam_z} 0 ${cam_pitch} 0</pose>
         <axis>
           <xyz>0 0 1</xyz>
