Commit message: feat: implement auto-driving wander node for SLAM bootstrapping; update launch files and documentation

File: vslam_description/urdf/gz_slim_tb3.sdf.xacro (robot description, xacro)
@@ -35,5 +35,9 @@
     <!-- negative pitch = nose up in SDF -->
     <xacro:property name="cam_pitch" value="-0.0873"/>
-    <xacro:property name="mast_x" value="0.010"/>
+    <!-- Camera shares the lidar's post (x=-0.032) instead of sitting on its
+         own forward bracket - mounted directly above/behind the lidar on the
+         same mast. Both are well clear of each other in z (0.150 vs 0.250),
+         so the camera housing does not occlude the lidar's scan plane. -->
+    <xacro:property name="sensor_post_x" value="-0.032"/>
     <!-- colour scheme -->
     <xacro:property name="c_body" value="0.10 0.28 0.32"/>
@@ -82,12 +86,12 @@
           </material>
         </visual>
-        <!-- camera mast -->
-        <!-- post carrying the lidar above the camera bracket -->
-        <visual name="lidar_post_visual">
-          <pose>-0.032 0 ${(deck_z + 0.150) / 2} 0 0 0</pose>
+        <!-- Single post carrying both the lidar (partway up) and the camera
+             (on top, directly behind/above the lidar) - see sensor_post_x. -->
+        <visual name="sensor_post_visual">
+          <pose>${sensor_post_x} 0 ${(deck_z + cam_z) / 2} 0 0 0</pose>
           <geometry>
             <cylinder>
               <radius>0.010</radius>
-              <length>${0.150 - deck_z}</length>
+              <length>${cam_z - deck_z}</length>
             </cylinder>
           </geometry>
@@ -97,22 +101,10 @@
           </material>
         </visual>
-        <visual name="mast_visual">
-          <pose>${mast_x} 0 ${(deck_z + cam_z) / 2} 0 0 0</pose>
+        <!-- small mounting cap connecting the post top to the camera housing -->
+        <visual name="camera_mount_visual">
+          <pose>${sensor_post_x} 0 ${cam_z} 0 ${cam_pitch} 0</pose>
           <geometry>
             <box>
-              <size>0.016 0.030 ${cam_z - deck_z}</size>
-            </box>
-          </geometry>
-          <material>
-            <ambient>0.05 0.05 0.06 1</ambient>
-            <diffuse>${c_dark} 1</diffuse>
-          </material>
-        </visual>
-        <!-- bracket arm from mast to camera -->
-        <visual name="mast_arm_visual">
-          <pose>${(mast_x + 0.032) / 2} 0 ${cam_z} 0 ${cam_pitch} 0</pose>
-          <geometry>
-            <box>
-              <size>0.030 0.024 0.008</size>
+              <size>0.024 0.024 0.008</size>
             </box>
           </geometry>
@@ -385,10 +377,10 @@
         </collision>
       </link>
-      <!-- forward monocular camera, centred on y, at the height the lidar
-           tower used to occupy. 480x480 @ 30 Hz.
+      <!-- forward monocular camera, centred on y, mounted directly above/
+           behind the lidar on the shared sensor post. 480x480 @ 30 Hz.
            Measured intrinsics: fx = fy = 415.787, cx = cy = 240.
            These MUST stay in sync with vslam_slam/config/tb3.yaml. -->
       <link name="camera_link">
-        <pose>0.032 0 ${cam_z} 0 ${cam_pitch} 0</pose>
+        <pose>${sensor_post_x} 0 ${cam_z} 0 ${cam_pitch} 0</pose>
         <inertial>
           <pose>0 0 0 0 0 0</pose>
@@ -482,5 +474,5 @@
         <parent>base_link</parent>
         <child>camera_link</child>
-        <pose>0.032 0 ${cam_z} 0 ${cam_pitch} 0</pose>
+        <pose>${sensor_post_x} 0 ${cam_z} 0 ${cam_pitch} 0</pose>
         <axis>
           <xyz>0 0 1</xyz>

Commit message: feat: enhance navigation parameters and documentation; separate lidar and camera mounts for improved SLAM performance

File: vslam_description/urdf/gz_slim_tb3.sdf.xacro (robot description, xacro)
@@ -29,15 +29,20 @@
          low-parallax, repetitively textured, and a poor diet for monocular
          tracking. At 0.25 with a 5 deg upward tilt the floor starts ~0.7 m out
-         and pillars/walls dominate the frame.
-         The lidar scan plane is at 0.150; the bracket crossing it sits 0.061 m
-         from the lidar, inside range_min 0.12, so it is not seen. -->
+         and pillars/walls dominate the frame. -->
     <xacro:property name="cam_z" value="0.250"/>
     <!-- negative pitch = nose up in SDF -->
     <xacro:property name="cam_pitch" value="-0.0873"/>
-    <!-- Camera shares the lidar's post (x=-0.032) instead of sitting on its
-         own forward bracket - mounted directly above/behind the lidar on the
-         same mast. Both are well clear of each other in z (0.150 vs 0.250),
-         so the camera housing does not occlude the lidar's scan plane. -->
-    <xacro:property name="sensor_post_x" value="-0.032"/>
+    <!-- Lidar and camera are on SEPARATE masts, not stacked coaxially. A
+         stacked design (one post through the lidar's z-extent, or two
+         segments dodging around it) always leaves a single rod running
+         through the same x,y point as the lidar body - not something you can
+         actually build. Real mounts sit side by side instead.
+         Lidar mounts flush on the deck (x=-0.032, matches its own link pose)
+         at real hardware height; camera_post_x is offset far enough behind it
+         (more negative x) to clear the lidar's 0.0508 m radius with margin:
+         separation 0.068 m > (0.0508 lidar + 0.010 post) = 0.0608 m
+         required, i.e. 7.2mm clearance. Verified no lateral overlap at any
+         height. -->
+    <xacro:property name="camera_post_x" value="-0.10"/>
     <!-- colour scheme -->
     <xacro:property name="c_body" value="0.10 0.28 0.32"/>
@@ -86,8 +91,9 @@
           </material>
         </visual>
-        <!-- Single post carrying both the lidar (partway up) and the camera
-             (on top, directly behind/above the lidar) - see sensor_post_x. -->
-        <visual name="sensor_post_visual">
-          <pose>${sensor_post_x} 0 ${(deck_z + cam_z) / 2} 0 0 0</pose>
+        <!-- Camera's own mast, a single straight post from the deck up to the
+             camera. Offset in x from the lidar (camera_post_x, see above) so
+             it never crosses the lidar's body, at any height. -->
+        <visual name="camera_post_visual">
+          <pose>${camera_post_x} 0 ${(deck_z + cam_z) / 2} 0 0 0</pose>
           <geometry>
             <cylinder>
@@ -103,5 +109,5 @@
         <!-- small mounting cap connecting the post top to the camera housing -->
         <visual name="camera_mount_visual">
-          <pose>${sensor_post_x} 0 ${cam_z} 0 ${cam_pitch} 0</pose>
+          <pose>${camera_post_x} 0 ${cam_z} 0 ${cam_pitch} 0</pose>
           <geometry>
             <box>
@@ -115,9 +121,13 @@
         </visual>
       </link>
-      <!-- LDS lidar for Nav2 costmaps. Mounted at z=0.150 on a post so it
-           clears the camera bracket (top at z=0.119) - a lower mount would
-           put the bracket in the scan and blind the robot forward. -->
+      <!-- LDS lidar, mounted flush on the deck like the real hardware - no
+           elevation needed once it is not sharing a mast with the camera.
+           Height is deck_z + half the lidar body (0.0275), sitting the lidar
+           body directly on the deck surface with no gap.
+           The camera's mast (at camera_post_x, offset sideways) does cross
+           the lidar's scan height, but only in a narrow arc directly behind
+           it - a small blind spot from the mount, same as real hardware. -->
       <link name="base_scan">
-        <pose>-0.032 0 0.150 0 0 0</pose>
+        <pose>-0.032 0 0.0875 0 0 0</pose>
         <inertial>
           <inertia>
@@ -382,5 +392,5 @@
            These MUST stay in sync with vslam_slam/config/tb3.yaml. -->
       <link name="camera_link">
-        <pose>${sensor_post_x} 0 ${cam_z} 0 ${cam_pitch} 0</pose>
+        <pose>${camera_post_x} 0 ${cam_z} 0 ${cam_pitch} 0</pose>
         <inertial>
           <pose>0 0 0 0 0 0</pose>
@@ -461,5 +471,5 @@
         <parent>base_link</parent>
         <child>base_scan</child>
-        <pose>-0.032 0 0.150 0 0 0</pose>
+        <pose>-0.032 0 0.0875 0 0 0</pose>
         <axis>
           <xyz>0 0 1</xyz>
@@ -474,5 +484,5 @@
         <parent>base_link</parent>
         <child>camera_link</child>
-        <pose>${sensor_post_x} 0 ${cam_z} 0 ${cam_pitch} 0</pose>
+        <pose>${camera_post_x} 0 ${cam_z} 0 ${cam_pitch} 0</pose>
         <axis>
           <xyz>0 0 1</xyz>
